File: shirasu.brd (EAGLE design)
At the start: 100 x 50 mm, 101 parts, among them J1 XT60PW-F, J2 XT60PW-M, J3 EP2.5-4-SIDE, J4 EP2.5-4-SIDE, J5 RJHSE-5381-02, J6 10118192-0001LF, Q1 TPH1R405PL,L1Q, Q2 TPH1R405PL,L1Q, Q3 TPH1R405PL,L1Q, Q4 TPH1R405PL,L1Q, U1 STM32F302_303C2, U10 MC34063AD, U11 INA2181A1IDGSR, U12 CSTNE_GH5L, U2 NCV7351D1E, U3 SI8621EC-B-IS, U4 TLP291, U5 BSS138BK, U6 MIC4606-2YTS-TR, U7 78L12F, U8 78L05F, U9 XC6206

Commit message: ver1.2
Parts:
- R39: value 10k -> 1k
- R40: value 1k -> 10k
- moved R39 3.13 mm to (56.8, 39.9), turned to 0 degrees
- moved R40 3.13 mm to (57.7, 42.9), turned to 90 degrees
Connections:
- net GNDA: now also R39.1; no longer R40.1
- net ISENSEB: now also U1.15; no longer U1.14
- net VCC: now also R40.2; no longer R39.2
- net VSENSE: now also R39.2, R40.1; no longer R39.1, R40.2
Other:
- board text added: "ver1.2"
- board text removed: "ver1.1"
Changed lines of the file:
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@@
 <setting verticaltext="up"/>
 </settings>
-<grid distance="10" unitdist="mm" unit="mm" style="lines" multiple="1" display="no" altdistance="5" altunitdist="mil" altunit="mil"/>
+<grid distance="1" unitdist="mm" unit="mm" style="lines" multiple="1" display="no" altdistance="5" altunitdist="mil" altunit="mil"/>
 <layers>
 <layer number="1" name="Top" color="4" fill="1" visible="yes" active="yes"/>
@@
 <wire x1="62.226" y1="17.674" x2="64.258" y2="17.674" width="0.1524" layer="22"/>
 <wire x1="64.258" y1="17.674" x2="66.29" y2="17.674" width="0.1524" layer="22"/>
-<text x="16.8" y="40.1" size="1.778" layer="21">ver1.1</text>
+<text x="16.8" y="40.1" size="1.778" layer="21">ver1.2</text>
 <text x="0" y="-0.15" size="0.06" layer="21" font="vector">C:/Users/ryuni/Desktop/python_workspace/image_th.bmp</text>
 <rectangle x1="14.575" y1="42.225" x2="14.825" y2="42.275" layer="21"/>
@@
 <attribute name="SPICEPREFIX" value="R" x="103.8" y="-75.89" size="1.778" layer="27" display="off"/>
 </element>
-<element name="R39" library="rcl" library_urn="urn:adsk.eagle:library:334" package="R0603" package3d_urn="urn:adsk.eagle:package:23555/3" value="10k" x="57.71" y="42.89" smashed="yes" rot="R90">
-<attribute name="NAME" x="55.275" y="39.155" size="1.27" layer="25" rot="R90"/>
+<element name="R40" library="rcl" library_urn="urn:adsk.eagle:library:334" package="R0603" package3d_urn="urn:adsk.eagle:package:23555/3" value="10k" x="57.71" y="42.89" smashed="yes" rot="R90">
+<attribute name="NAME" x="54.155" y="41.725" size="1.016" layer="25"/>
 <attribute name="POPULARITY" value="70" x="155.5" y="84.8" size="1.778" layer="27" rot="R90" display="off"/>
 <attribute name="SPICEPREFIX" value="R" x="155.5" y="84.8" size="1.778" layer="27" rot="R90" display="off"/>
 </element>
-<element name="R40" library="rcl" library_urn="urn:adsk.eagle:library:334" package="R0603" package3d_urn="urn:adsk.eagle:package:23555/3" value="1k" x="56.81" y="39.89" smashed="yes">
-<attribute name="NAME" x="57.175" y="40.975" size="1.27" layer="25" rot="R90"/>
+<element name="R39" library="rcl" library_urn="urn:adsk.eagle:library:334" package="R0603" package3d_urn="urn:adsk.eagle:package:23555/3" value="1k" x="56.81" y="39.89" smashed="yes">
+<attribute name="NAME" x="55.025" y="41.175" size="1.27" layer="25" rot="R180"/>
 <attribute name="POPULARITY" value="70" x="103.8" y="-57.9" size="1.778" layer="27" display="off"/>
 <attribute name="SPICEPREFIX" value="R" x="103.8" y="-57.9" size="1.778" layer="27" display="off"/>
@@
 <contactref element="J4" pad="1"/>
 <contactref element="C38" pad="1"/>
-<contactref element="R40" pad="1"/>
+<contactref element="R39" pad="1"/>
 <contactref element="C30" pad="1"/>
 <contactref element="C33" pad="1"/>
@@
 <contactref element="U10" pad="6"/>
 <contactref element="C7" pad="1"/>
-<contactref element="R39" pad="2"/>
+<contactref element="R40" pad="2"/>
 <contactref element="U7" pad="3"/>
 <wire x1="63.581" y1="43.199" x2="66.059" y2="43.199" width="0.254" layer="1"/>
@@
 </signal>
 <signal name="VSENSE">
-<contactref element="R39" pad="1"/>
-<contactref element="R40" pad="2"/>
+<contactref element="R40" pad="1"/>
+<contactref element="R39" pad="2"/>
 <contactref element="C30" pad="2"/>
 <contactref element="U1" pad="10"/>
@@
 <contactref element="R37" pad="2"/>
 <contactref element="C39" pad="2"/>
-<contactref element="U1" pad="14"/>
 <contactref element="U1" pad="13"/>
 <wire x1="69.83" y1="25.05" x2="71.1709125" y2="25.05" width="0.1524" layer="1"/>
-<wire x1="71.1709125" y1="25.05" x2="71.87801875" y2="25.05" width="0.1524" layer="1"/>
-<wire x1="71.87801875" y1="25.05" x2="72.353803125" y2="25.525784375" width="0.1524" layer="1"/>
 <wire x1="72.00025" y1="25.8793375" x2="71.1709125" y2="25.05" width="0.1524" layer="1"/>
 <wire x1="67.9" y1="24.14" x2="68.14" y2="24.14" width="0.1524" layer="1"/>
 <wire x1="68.14" y1="24.14" x2="69.05" y2="25.05" width="0.1524" layer="1"/>
 <wire x1="69.05" y1="25.05" x2="69.83" y2="25.05" width="0.1524" layer="1"/>
+<contactref element="U1" pad="15"/>
+<wire x1="71.944803125" y1="24.76735625" x2="71.662159375" y2="25.05" width="0.1524" layer="1"/>
+<wire x1="71.662159375" y1="25.05" x2="71.1709125" y2="25.05" width="0.1524" layer="1"/>
+<wire x1="72.70735625" y1="25.17223125" x2="72.30248125" y2="24.76735625" width="0.1524" layer="1"/>
+<wire x1="72.30248125" y1="24.76735625" x2="71.944803125" y2="24.76735625" width="0.1524" layer="1"/>
 </signal>
 <signal name="BOOT0">
